Commit message: Migration to Jazzy

File: src/mowerai/description/mower.urdf.xacro (robot description, xacro)
@@ -2,4 +2,5 @@
 <robot xmlns:xacro="http://www.ros.org/wiki/xacro" name="mower">
    <xacro:include filename="include.xacro" />
+   <xacro:include filename="inertial_macros.xacro" />
    <link name="world"></link>
    <joint name="base_joint" type="fixed">
@@ -24,25 +25,31 @@
             </geometry>
         </collision>
-        <inertial>
+        <xacro:inertial_box mass="0.5" x="0.9144" y="0.6096" z="0.03175">
             <origin xyz="0 0 0.05" rpy="0 0 0"/>
-            <mass value="12" />
-            <inertia ixx="2.26" ixy="0.0" ixz="0.0" iyy="6.26" iyz="0.0" izz="8.5" />
-        </inertial>
+        </xacro:inertial_box>
     </link>
     <joint name="wheel_fr_joint" type="continuous">
-        <origin xyz="0.4572 0.3048 0" rpy="0 0 0"/>
+        <origin xyz="0.4572 0.3048 0" rpy="${pi/2} 0 0"/>
+        <axis xyz="0 0 -1"/>
         <parent link="base_link"/>
+        <child link="wheel_fr_link"/>
     </joint>
     <joint name="wheel_fl_joint" type="continuous">
-        <origin xyz="0.4572 0.3048 0" rpy="0 0 0"/>
+        <origin xyz="0.4572 0.3048 0" rpy="-${pi/2} 0 0"/>
+        <axis xyz="0 0 1"/>
         <parent link="base_link"/>
+        <child link="wheel_fl_link"/>
     </joint>
     <joint name="wheel_rr_joint" type="continuous">
-        <origin xyz="0.4572 0.3048 0" rpy="0 0 0"/>
+        <origin xyz="0.4572 0.3048 0" rpy="${pi/2} 0 0"/>
+        <axis xyz="0 0 -1"/>
         <parent link="base_link"/>
+        <child link="wheel_rr_link"/>
     </joint>
     <joint name="wheel_rl_joint" type="continuous">
-        <origin xyz="0.4572 0.3048 0" rpy="0 0 0"/>
+        <origin xyz="0.4572 0.3048 0" rpy="-${pi/2} 0 0"/>
+        <axis xyz="0 0 1"/>
         <parent link="base_link"/>
+        <child link="wheel_rl_link"/>
     </joint>
     <link name="wheel_fr_link">
@@ -50,5 +57,5 @@
             <origin xyz="0 0 0" rpy="0 0 0"/>
             <geometry>
-                <cylinder size="2.5 1.5 0.1" />
+                <cylinder length="0.0508" radius="0.1016" />
             </geometry>
             <material name="green">
@@ -59,5 +66,5 @@
             <origin xyz="0 0 0" rpy="0 0 0"/>
             <geometry>
-                <cylinder size="2.5 1.5 0.1" />
+                <cylinder length="0.0508" radius="0.1016" />
             </geometry>
         </collision>
@@ -72,5 +79,5 @@
             <origin xyz="0 0 0" rpy="0 0 0"/>
             <geometry>
-                <cylinder size="2.5 1.5 0.1" />
+                <cylinder length="0.0508" radius="0.1016" />
             </geometry>
             <material name="green">
@@ -81,5 +88,5 @@
             <origin xyz="0 0 0" rpy="0 0 0"/>
             <geometry>
-                <cylinder size="2.5 1.5 0.1" />
+                <cylinder length="0.0508" radius="0.1016" />
             </geometry>
         </collision>
@@ -94,5 +101,5 @@
             <origin xyz="0 0 0" rpy="0 0 0"/>
             <geometry>
-                <cylinder size="2.5 1.5 0.1" />
+                <cylinder length="0.0508" radius="0.1016" />
             </geometry>
             <material name="green">
@@ -103,5 +110,5 @@
             <origin xyz="0 0 0" rpy="0 0 0"/>
             <geometry>
-                <cylinder size="2.5 1.5 0.1" />
+                <cylinder length="0.0508" radius="0.1016" />
             </geometry>
         </collision>
@@ -116,5 +123,5 @@
             <origin xyz="0 0 0" rpy="0 0 0"/>
             <geometry>
-                <cylinder size="2.5 1.5 0.1" />
+                <cylinder length="0.0508" radius="0.1016" />
             </geometry>
             <material name="green">
@@ -125,5 +132,5 @@
             <origin xyz="0 0 0" rpy="0 0 0"/>
             <geometry>
-                <cylinder size="2.5 1.5 0.1" />
+                <cylinder length="0.0508" radius="0.1016" />
             </geometry>
         </collision>
